File: eagle/robogram.sch (EAGLE design)
At the start: 7 parts, among them IC1 ATMEGA328-20P, Q1 14.7456MHz

Commit message: getting set up for deving
Parts:
- added ISP1: AVRISP-6, adafruit:AVRISP-6
- added JP1, JP2: (no value), adafruit:PINHD-1X8BIG
- added LED1: (no value), adafruit:LED3MM
- added R1: 10k, adafruit:R-US_0204/5
- added R2: (no value), adafruit:R-US_0204/5
- added S2: DTE6K, switch-misc:DTE6K
Connections:
- new net N$10: IC1.(PCI19/INT1/OC2B)PD3, JP1.4
- new net N$11: IC1.(PCI20/XCK/T0)PD4, JP1.5
- new net N$12: IC1.(PCI21/T1/OC0B)PD5, JP1.6
- new net N$13: IC1.(PCI22/AIN0OC0A)PD6, JP1.7
- new net N$14: IC1.(PCI23/AIN1)PD7, JP1.8
- new net N$15: IC1.(PCI2/SS/OC1B)PB2, R2.1
- new net N$16: LED1.A, R2.2
- new net N$17: IC1.(PCI1/OC1A/OC1S)PB1, JP2.2
- new net N$18: IC1.(PCI0/ICP/CLKO)PB0, JP2.1
- new net N$19: IC1.(PCI8/ADC0)PC0, JP2.3
- new net N$20: IC1.(PCI9/ADC1)PC1, JP2.4
- new net N$21: IC1.(PCI10/ADC2)PC2, JP2.5
- new net N$22: IC1.(PCI11/ADC3)PC3, JP2.6
- new net N$23: IC1.(PCI12/ADC4/SDA)PC4, JP2.7
- new net N$24: IC1.(PCI13/ADC5/SCL)PC5, JP2.8
- new net N$3: IC1.PC6(/RESET/PCI14), ISP1.RST, R1.2, S2.S
- new net N$4: IC1.(PCI3/MOSI/OC2A)PB3, ISP1.MOSI
- new net N$5: IC1.(PCI4/MISO)PB4, ISP1.MISO
- new net N$6: IC1.(PCI5/SCK)PB5, ISP1.SCK
- new net N$7: IC1.(PCI16/RXD)PD0, JP1.1
- new net N$8: IC1.(PCI17/TXD)PD1, JP1.2
- new net N$9: IC1.(PCI18/INT0)PD2, JP1.3
- net GND: now also ISP1.GND, LED1.C, S2.P
- net VCC: now also ISP1.VCC, R1.1
